Commit message: Changed Gazebo mesh colors, changed to position based control for simulation

File: franka_description/robots/panda.gazebo.xacro (robot description, xacro)
@@ -4,5 +4,5 @@
         <!-- Link0 -->
         <gazebo reference="${robot_name}_link0">
-            <material>Gazebo/Grey</material>
+            <!-- <material>Gazebo/Grey</material> -->
             <mu1>0.2</mu1>
             <mu2>0.2</mu2>
@@ -10,5 +10,5 @@
         <!-- Link1 -->
         <gazebo reference="${robot_name}_link1">
-            <material>Gazebo/White</material>
+            <!-- <material>Gazebo/White</material> -->
             <mu1>0.2</mu1>
             <mu2>0.2</mu2>
@@ -16,5 +16,5 @@
         <!-- Link2 -->
         <gazebo reference="${robot_name}_link2">
-            <material>Gazebo/White</material>
+            <!-- <material>Gazebo/White</material> -->
             <mu1>0.2</mu1>
             <mu2>0.2</mu2>
@@ -22,5 +22,5 @@
         <!-- Link3 -->
         <gazebo reference="${robot_name}_link3">
-            <material>Gazebo/White</material>
+            <!-- <material>Gazebo/White</material> -->
             <mu1>0.2</mu1>
             <mu2>0.2</mu2>
@@ -28,5 +28,5 @@
         <!-- Link4 -->
         <gazebo reference="${robot_name}_link4">
-            <material>Gazebo/White</material>
+            <!-- <material>Gazebo/White</material> -->
             <mu1>0.2</mu1>
             <mu2>0.2</mu2>
@@ -34,5 +34,5 @@
         <!-- Link5 -->
         <gazebo reference="${robot_name}_link5">
-            <material>Gazebo/White</material>
+            <!-- <material>Gazebo/White</material> -->
             <mu1>0.2</mu1>
             <mu2>0.2</mu2>
@@ -40,5 +40,5 @@
         <!-- Link6 -->
         <gazebo reference="${robot_name}_link6">
-            <material>Gazebo/White</material>
+            <!-- <material>Gazebo/White</material> -->
             <mu1>0.2</mu1>
             <mu2>0.2</mu2>
@@ -46,5 +46,5 @@
         <!-- Link7 -->
         <gazebo reference="${robot_name}_link7">
-            <material>Gazebo/Grey</material>
+            <!-- <material>Gazebo/Grey</material> -->
             <mu1>0.2</mu1>
             <mu2>0.2</mu2>
@@ -52,5 +52,5 @@
         <!-- Link8 -->
         <gazebo reference="${robot_name}_link8">
-            <material>Gazebo/Grey</material>
+            <!-- <material>Gazebo/Grey</material> -->
             <mu1>0.2</mu1>
             <mu2>0.2</mu2>
@@ -58,5 +58,5 @@
         <!-- LinkHand -->
         <gazebo reference="${robot_name}_hand">
-            <material>Gazebo/Grey</material>
+            <!-- <material>Gazebo/Grey</material> -->
             <mu1>0.2</mu1>
             <mu2>0.2</mu2>
@@ -64,5 +64,5 @@
         <!-- LinkRightFinger -->
         <gazebo reference="${robot_name}_rightfinger">
-            <material>Gazebo/Grey</material>
+            <!-- <material>Gazebo/Grey</material> -->
             <mu1>0.2</mu1>
             <mu2>0.2</mu2>
@@ -70,5 +70,5 @@
         <!-- LinkLeftFinger -->
         <gazebo reference="${robot_name}_leftfinger">
-            <material>Gazebo/Grey</material>
+            <!-- <material>Gazebo/Grey</material> -->
             <mu1>0.2</mu1>
             <mu2>0.2</mu2>
