Commit message: Modifications to use either position or effort controllers

File: franka_description/robots/panda_arm_hand.urdf.xacro (robot description, xacro)
@@ -1,26 +1,33 @@
 <?xml version="1.0" encoding="utf-8"?>
 <robot xmlns:xacro="http://www.ros.org/wiki/xacro" name="panda">
-  <!-- Initialize xacro parameters -->
-  <xacro:arg name="robot_name" default="panda"/>
-  <!-- Initialize gripper_center properties -->
-  <xacro:arg name="gripper_center" default="false" />
-  <xacro:property name="gripper_center" value="$(arg gripper_center)"/>
-  <xacro:arg name="gripper_center_xyz" default="0.0 0.0 0.10" />
-  <xacro:property name="gripper_center_xyz" value="$(arg gripper_center_xyz)"/>
-  <xacro:arg name="gripper_center_rpy" default="0.0 0.0 0.0" />
-  <xacro:property name="gripper_center_rpy" value="$(arg gripper_center_rpy)"/>
-  <!-- Include xacro files -->
-  <xacro:include filename="$(find franka_description)/robots/panda_arm.xacro"/>
-  <xacro:include filename="$(find franka_description)/robots/hand.xacro"/>
-  <!-- for simulation -->
-  <xacro:include filename="$(find franka_description)/robots/panda.gazebo.xacro"/>
-  <xacro:include filename="$(find franka_description)/robots/panda.transmission.xacro"/>
-  <!-- end for simulation -->
-  <!-- Generate urdfs -->
-  <xacro:panda_arm />
-  <xacro:hand ns="panda" rpy="0 0 ${-pi/4}" connected_to="panda_link8" gripper_center="${gripper_center}" gripper_center_xyz="${gripper_center_xyz}" gripper_center_rpy="${gripper_center_rpy}"/>
-  <!-- for simulation -->
-  <xacro:panda_gazebo robot_name="$(arg robot_name)" />
-  <xacro:panda_transmission robot_name="$(arg robot_name)" load_hand="true"/>
-  <!-- end for simulation -->
+    <!-- Initialize xacro parameters -->
+    <xacro:arg name="robot_name" default="panda"/>
+    <xacro:arg name="controller_type" default="position"/>
+    <xacro:property name="controller_type" value="$(arg controller_type)"/>
+    <!-- Initialize gripper_center properties -->
+    <xacro:arg name="gripper_center" default="false" />
+    <xacro:property name="gripper_center" value="$(arg gripper_center)"/>
+    <xacro:arg name="gripper_center_xyz" default="0.0 0.0 0.10" />
+    <xacro:property name="gripper_center_xyz" value="$(arg gripper_center_xyz)"/>
+    <xacro:arg name="gripper_center_rpy" default="0.0 0.0 0.0" />
+    <xacro:property name="gripper_center_rpy" value="$(arg gripper_center_rpy)"/>
+    <!-- Include xacro files -->
+    <xacro:include filename="$(find franka_description)/robots/panda_arm.xacro"/>
+    <xacro:include filename="$(find franka_description)/robots/hand.xacro"/>
+    <!-- for simulation -->
+    <xacro:include filename="$(find franka_description)/robots/panda.gazebo.xacro"/>
+    <xacro:if value="${controller_type == 'position'}">
+        <xacro:include filename="$(find franka_description)/robots/panda.transmission.position.xacro"/>
+    </xacro:if>
+    <xacro:if value="${controller_type == 'effort'}">
+        <xacro:include filename="$(find franka_description)/robots/panda.transmission.effort.xacro"/>
+    </xacro:if>
+    <!-- end for simulation -->
+    <!-- Generate urdfs -->
+    <xacro:panda_arm />
+    <xacro:hand ns="panda" rpy="0 0 ${-pi/4}" connected_to="panda_link8" gripper_center="${gripper_center}" gripper_center_xyz="${gripper_center_xyz}" gripper_center_rpy="${gripper_center_rpy}"/>
+    <!-- for simulation -->
+    <xacro:panda_gazebo robot_name="$(arg robot_name)" />
+    <xacro:panda_transmission robot_name="$(arg robot_name)" load_hand="true"/>
+    <!-- end for simulation -->
 </robot>
