Commit message: parametrize controllers

File: franka_description/robots/panda.transmission.xacro (robot description, xacro)
@@ -2,4 +2,10 @@
 <robot xmlns:xacro="http://www.ros.org/wiki/xacro">
     <xacro:macro name="panda_transmission" params="robot_name load_hand">
+        <xacro:macro name="pandaArmHardwareInterface">
+            <hardwareInterface>hardware_interface/PositionJointInterface</hardwareInterface>
+        </xacro:macro>
+        <xacro:macro name="pandaHandHardwareInterface">
+            <hardwareInterface>hardware_interface/PositionJointInterface</hardwareInterface>
+        </xacro:macro>
         <!-- Load Gazebo lib and set the robot namespace -->
         <gazebo>
@@ -11,8 +17,8 @@
             <type>transmission_interface/SimpleTransmission</type>
             <joint name="${robot_name}_joint1">
-                <hardwareInterface>hardware_interface/PositionJointInterface</hardwareInterface>
+                <xacro:pandaArmHardwareInterface/>
             </joint>
             <actuator name="${robot_name}_motor_1">
-                <hardwareInterface>hardware_interface/PositionJointInterface</hardwareInterface>
+                <xacro:pandaArmHardwareInterface/>
                 <mechanicalReduction>1</mechanicalReduction>
             </actuator>
@@ -21,8 +27,8 @@
             <type>transmission_interface/SimpleTransmission</type>
             <joint name="${robot_name}_joint2">
-                <hardwareInterface>hardware_interface/PositionJointInterface</hardwareInterface>
+                <xacro:pandaArmHardwareInterface/>
             </joint>
             <actuator name="${robot_name}_motor_2">
-                <hardwareInterface>hardware_interface/PositionJointInterface</hardwareInterface>
+                <xacro:pandaArmHardwareInterface/>
                 <mechanicalReduction>1</mechanicalReduction>
             </actuator>
@@ -31,8 +37,8 @@
             <type>transmission_interface/SimpleTransmission</type>
             <joint name="${robot_name}_joint3">
-                <hardwareInterface>hardware_interface/PositionJointInterface</hardwareInterface>
+                <xacro:pandaArmHardwareInterface/>
             </joint>
             <actuator name="${robot_name}_motor_3">
-                <hardwareInterface>hardware_interface/PositionJointInterface</hardwareInterface>
+                <xacro:pandaArmHardwareInterface/>
                 <mechanicalReduction>1</mechanicalReduction>
             </actuator>
@@ -41,8 +47,8 @@
             <type>transmission_interface/SimpleTransmission</type>
             <joint name="${robot_name}_joint4">
-                <hardwareInterface>hardware_interface/PositionJointInterface</hardwareInterface>
+                <xacro:pandaArmHardwareInterface/>
             </joint>
             <actuator name="${robot_name}_motor_4">
-                <hardwareInterface>hardware_interface/PositionJointInterface</hardwareInterface>
+                <xacro:pandaArmHardwareInterface/>
                 <mechanicalReduction>1</mechanicalReduction>
             </actuator>
@@ -51,8 +57,8 @@
             <type>transmission_interface/SimpleTransmission</type>
             <joint name="${robot_name}_joint5">
-                <hardwareInterface>hardware_interface/PositionJointInterface</hardwareInterface>
+                <xacro:pandaArmHardwareInterface/>
             </joint>
             <actuator name="${robot_name}_motor_5">
-                <hardwareInterface>hardware_interface/PositionJointInterface</hardwareInterface>
+                <xacro:pandaArmHardwareInterface/>
                 <mechanicalReduction>1</mechanicalReduction>
             </actuator>
@@ -61,8 +67,8 @@
             <type>transmission_interface/SimpleTransmission</type>
             <joint name="${robot_name}_joint6">
-                <hardwareInterface>hardware_interface/PositionJointInterface</hardwareInterface>
+                <xacro:pandaArmHardwareInterface/>
             </joint>
             <actuator name="${robot_name}_motor_6">
-                <hardwareInterface>hardware_interface/PositionJointInterface</hardwareInterface>
+                <xacro:pandaArmHardwareInterface/>
                 <mechanicalReduction>1</mechanicalReduction>
             </actuator>
@@ -71,8 +77,8 @@
             <type>transmission_interface/SimpleTransmission</type>
             <joint name="${robot_name}_joint7">
-                <hardwareInterface>hardware_interface/PositionJointInterface</hardwareInterface>
+                <xacro:pandaArmHardwareInterface/>
             </joint>
             <actuator name="${robot_name}_motor_7">
-                <hardwareInterface>hardware_interface/PositionJointInterface</hardwareInterface>
+                <xacro:pandaArmHardwareInterface/>
                 <mechanicalReduction>1</mechanicalReduction>
             </actuator>
@@ -82,8 +88,8 @@
                 <type>transmission_interface/SimpleTransmission</type>
                 <joint name="${robot_name}_finger_joint1">
-                    <hardwareInterface>hardware_interface/PositionJointInterface</hardwareInterface>
+                    <xacro:pandaHandHardwareInterface/>
                 </joint>
                 <actuator name="${robot_name}_finger_joint1">
-                    <hardwareInterface>hardware_interface/PositionJointInterface</hardwareInterface>
+                    <xacro:pandaHandHardwareInterface/>
                     <mechanicalReduction>1</mechanicalReduction>
                 </actuator>
@@ -92,8 +98,8 @@
                 <type>transmission_interface/SimpleTransmission</type>
                 <joint name="${robot_name}_finger_joint2">
-                    <hardwareInterface>hardware_interface/PositionJointInterface</hardwareInterface>
+                    <xacro:pandaHandHardwareInterface/>
                 </joint>
                 <actuator name="${robot_name}_finger_joint2">
-                    <hardwareInterface>hardware_interface/PositionJointInterface</hardwareInterface>
+                    <xacro:pandaHandHardwareInterface/>
                     <mechanicalReduction>1</mechanicalReduction>
                 </actuator>
