Commit message: Add new parameters

File: franka_description/robots/panda_arm.xacro (robot description, xacro)
@@ -49,9 +49,11 @@
       </collision>
       <!-- for simulation -->
-      <inertial>
-        <origin xyz="0 0 0" rpy="0 0 0" />
-        <mass value="2.34" />
-        <inertia ixx="0.3" ixy="0.0" ixz="0.0" iyy="0.3" iyz="0.0" izz="0.3" />
-      </inertial>
+      <!-- Link 1 -->
+        <!-- Generated From:  git@github.com:marcocognetti/FrankaEmikaPandaDynModel.git -->
+        <inertial>
+            <origin xyz="-0.000828 0.004496 -0.292171" rpy="0 0 0" />
+            <mass value="1.654831"/>
+            <inertia  ixx="0.637949" ixy="0.000056" ixz="0.000613" iyy="0.637409" iyz="-0.021115" izz="0.001173"  />
+        </inertial>
       <!-- end for simulation -->
     </link>
@@ -79,9 +81,11 @@
       </collision>
       <!-- for simulation -->
-      <inertial>
-        <origin xyz="0 0 0" rpy="0 0 0" />
-        <mass value="2.36" />
-        <inertia ixx="0.3" ixy="0.0" ixz="0.0" iyy="0.3" iyz="0.0" izz="0.3" />
-      </inertial>
+        <!-- Link 2 -->
+        <!-- Generated From:  git@github.com:marcocognetti/FrankaEmikaPandaDynModel.git -->
+        <inertial>
+            <origin xyz="0.003569 -0.027131 -0.014413" rpy="0 0 0" />
+            <mass value="8.107980"/>
+            <inertia  ixx="0.024018" ixy="-0.003820" ixz="0.003154" iyy="0.016501" iyz="-0.012389" izz="0.025322"  />
+        </inertial>
       <!-- end for simulation -->
     </link>
@@ -109,9 +113,11 @@
       </collision>
       <!-- for simulation -->
-      <inertial>
-        <origin xyz="0 0 0" rpy="0 0 0" />
-        <mass value="2.38" />
-        <inertia ixx="0.3" ixy="0.0" ixz="0.0" iyy="0.3" iyz="0.0" izz="0.3" />
-      </inertial>
+        <!-- Link 3 -->
+        <!-- Generated From:  git@github.com:marcocognetti/FrankaEmikaPandaDynModel.git -->
+        <inertial>
+            <origin xyz="0.032833 -0.002029 -0.096799" rpy="0 0 0" />
+            <mass value="3.300138"/>
+            <inertia  ixx="0.035301" ixy="0.011494" ixz="-0.016618" iyy="0.003726" iyz="-0.013031" izz="0.000000"  />
+        </inertial>
       <!-- end for simulation -->
     </link>
@@ -139,9 +145,11 @@
       </collision>
       <!-- for simulation -->
-      <inertial>
-        <origin xyz="0 0 0" rpy="0 0 0" />
-        <mass value="2.43" />
-        <inertia ixx="0.3" ixy="0.0" ixz="0.0" iyy="0.3" iyz="0.0" izz="0.3" />
-      </inertial>
+        <!-- Link 4 -->
+        <!-- Generated From:  git@github.com:marcocognetti/FrankaEmikaPandaDynModel.git -->
+        <inertial>
+            <origin xyz="-0.043407 0.128195 0.002060" rpy="0 0 0" />
+            <mass value="2.548403"/>
+            <inertia  ixx="0.022739" ixy="-0.011128" ixz="0.003843" iyy="0.000000" iyz="0.007803" izz="0.028460"  />
+        </inertial>
       <!-- end for simulation -->
     </link>
@@ -169,9 +177,11 @@
       </collision>
       <!-- for simulation -->
-      <inertial>
-        <origin xyz="0 0 0" rpy="0 0 0" />
-        <mass value="3.5" />
-        <inertia ixx="0.3" ixy="0.0" ixz="0.0" iyy="0.3" iyz="0.0" izz="0.3" />
-      </inertial>
+        <!-- Link 5 -->
+        <!-- Generated From:  git@github.com:marcocognetti/FrankaEmikaPandaDynModel.git -->
+        <inertial>
+            <origin xyz="-0.000323 0.021146 -0.124488" rpy="0 0 0" />
+            <mass value="2.095362"/>
+            <inertia  ixx="0.025776" ixy="0.003369" ixz="-0.010502" iyy="0.034795" iyz="0.002025" izz="0.000000"  />
+        </inertial>
       <!-- end for simulation -->
     </link>
@@ -199,9 +209,11 @@
       </collision>
       <!-- for simulation -->
-      <inertial>
-        <origin xyz="0 0 0" rpy="0 0 0" />
-        <mass value="1.47" />
-        <inertia ixx="0.3" ixy="0.0" ixz="0.0" iyy="0.3" iyz="0.0" izz="0.3" />
-      </inertial>
+        <!-- Link 6 -->
+        <!-- Generated From:  git@github.com:marcocognetti/FrankaEmikaPandaDynModel.git -->
+        <inertial>
+            <origin xyz="0.066189 -0.018040 -0.021379" rpy="0 0 0" />
+            <mass value="1.722535"/>
+            <inertia  ixx="0.000104" ixy="-0.003459" ixz="0.002509" iyy="0.003188" iyz="0.001801" izz="0.000622"  />
+        </inertial>
       <!-- end for simulation -->
     </link>
@@ -229,9 +241,11 @@
       </collision>
       <!-- for simulation -->
-      <inertial>
-        <origin xyz="0 0 0" rpy="0 0 0" />
-        <mass value="0.45" />
-        <inertia ixx="0.3" ixy="0.0" ixz="0.0" iyy="0.3" iyz="0.0" izz="0.3" />
-      </inertial>
+        <!-- Link 7 -->
+        <!-- Generated From:  git@github.com:marcocognetti/FrankaEmikaPandaDynModel.git -->
+        <inertial>
+            <origin xyz="0.001859 0.007351 0.055465" rpy="0 0 0" />
+            <mass value="0.570636"/>
+            <inertia  ixx="0.002852" ixy="0.004632" ixz="0.002398" iyy="0.000000" iyz="-0.002696" izz="0.000000"  />
+        </inertial>
       <!-- end for simulation -->
     </link>

Commit message: Reverted back to original dynamic params

File: franka_description/robots/panda_arm.xacro (robot description, xacro)
@@ -9,5 +9,5 @@
       </joint>
     </xacro:unless>
-    <!-- for simulation -->
+    <xacro:property name="joint_damping" value="1.0"/>
     <link name="world" />
     <joint name="robot_to_world" type="fixed">
@@ -15,7 +15,6 @@
       <child link="${arm_id}_link0" />
       <origin xyz="0.0 0.0 0.0" rpy="0.0 0.0 0.0" />
-    </joint>
-    <xacro:property name="joint_damping" value="1.0"/>
-    <!-- end for simulation -->
+      <dynamics damping="${joint_damping}"/>
+    </joint>
     <link name="${arm_id}_link0">
       <visual>
@@ -29,11 +28,9 @@
         </geometry>
       </collision>
-      <!-- for simulation -->
-      <inertial>
-        <origin xyz="0 0 0" rpy="0 0 0" />
-        <mass value="3.06" />
-        <inertia ixx="0.3" ixy="0.0" ixz="0.0" iyy="0.3" iyz="0.0" izz="0.3" />
-      </inertial>
-      <!-- end for simulation -->
+      <inertial>
+        <origin xyz="0 0 0" rpy="0 0 0"/>
+        <mass value="3.06"/>
+        <inertia ixx="0.3" ixy="0.0" ixz="0.0" iyy="0.3" iyz="0.0" izz="0.3"/>
+      </inertial>
     </link>
     <link name="${arm_id}_link1">
@@ -48,13 +45,9 @@
         </geometry>
       </collision>
-      <!-- for simulation -->
-      <!-- Link 1 -->
-        <!-- Generated From:  git@github.com:marcocognetti/FrankaEmikaPandaDynModel.git -->
-        <inertial>
-            <origin xyz="-0.000828 0.004496 -0.292171" rpy="0 0 0" />
-            <mass value="1.654831"/>
-            <inertia  ixx="0.637949" ixy="0.000056" ixz="0.000613" iyy="0.637409" iyz="-0.021115" izz="0.001173"  />
-        </inertial>
-      <!-- end for simulation -->
+      <inertial>
+        <origin xyz="0 0 0" rpy="0 0 0"/>
+        <mass value="2.34"/>
+        <inertia ixx="0.3" ixy="0.0" ixz="0.0" iyy="0.3" iyz="0.0" izz="0.3"/>
+      </inertial>
     </link>
     <joint name="${arm_id}_joint1" type="revolute">
@@ -65,7 +58,5 @@
       <axis xyz="0 0 1"/>
       <limit effort="87" lower="-2.8973" upper="2.8973" velocity="2.1750"/>
-      <!-- for simulation -->
-      <dynamics damping="${joint_damping}"/>
-      <!-- end for simulation -->
+      <dynamics damping="${joint_damping}"/>
     </joint>
     <link name="${arm_id}_link2">
@@ -80,13 +71,9 @@
         </geometry>
       </collision>
-      <!-- for simulation -->
-        <!-- Link 2 -->
-        <!-- Generated From:  git@github.com:marcocognetti/FrankaEmikaPandaDynModel.git -->
-        <inertial>
-            <origin xyz="0.003569 -0.027131 -0.014413" rpy="0 0 0" />
-            <mass value="8.107980"/>
-            <inertia  ixx="0.024018" ixy="-0.003820" ixz="0.003154" iyy="0.016501" iyz="-0.012389" izz="0.025322"  />
-        </inertial>
-      <!-- end for simulation -->
+      <inertial>
+        <origin xyz="0 0 0" rpy="0 0 0"/>
+        <mass value="2.36"/>
+        <inertia ixx="0.3" ixy="0.0" ixz="0.0" iyy="0.3" iyz="0.0" izz="0.3"/>
+      </inertial>
     </link>
     <joint name="${arm_id}_joint2" type="revolute">
@@ -97,7 +84,5 @@
       <axis xyz="0 0 1"/>
       <limit effort="87" lower="-1.7628" upper="1.7628" velocity="2.1750"/>
-      <!-- for simulation -->
-      <dynamics damping="${joint_damping}"/>
-      <!-- end for simulation -->
+      <dynamics damping="${joint_damping}"/>
     </joint>
     <link name="${arm_id}_link3">
@@ -112,13 +97,9 @@
         </geometry>
       </collision>
-      <!-- for simulation -->
-        <!-- Link 3 -->
-        <!-- Generated From:  git@github.com:marcocognetti/FrankaEmikaPandaDynModel.git -->
-        <inertial>
-            <origin xyz="0.032833 -0.002029 -0.096799" rpy="0 0 0" />
-            <mass value="3.300138"/>
-            <inertia  ixx="0.035301" ixy="0.011494" ixz="-0.016618" iyy="0.003726" iyz="-0.013031" izz="0.000000"  />
-        </inertial>
-      <!-- end for simulation -->
+      <inertial>
+        <origin xyz="0 0 0" rpy="0 0 0"/>
+        <mass value="2.38"/>
+        <inertia ixx="0.3" ixy="0.0" ixz="0.0" iyy="0.3" iyz="0.0" izz="0.3"/>
+      </inertial>
     </link>
     <joint name="${arm_id}_joint3" type="revolute">
@@ -129,7 +110,5 @@
       <axis xyz="0 0 1"/>
       <limit effort="87" lower="-2.8973" upper="2.8973" velocity="2.1750"/>
-      <!-- for simulation -->
-      <dynamics damping="${joint_damping}"/>
-      <!-- end for simulation -->
+      <dynamics damping="${joint_damping}"/>
     </joint>
     <link name="${arm_id}_link4">
@@ -144,13 +123,9 @@
         </geometry>
       </collision>
-      <!-- for simulation -->
-        <!-- Link 4 -->
-        <!-- Generated From:  git@github.com:marcocognetti/FrankaEmikaPandaDynModel.git -->
-        <inertial>
-            <origin xyz="-0.043407 0.128195 0.002060" rpy="0 0 0" />
-            <mass value="2.548403"/>
-            <inertia  ixx="0.022739" ixy="-0.011128" ixz="0.003843" iyy="0.000000" iyz="0.007803" izz="0.028460"  />
-        </inertial>
-      <!-- end for simulation -->
+      <inertial>
+        <origin xyz="0 0 0" rpy="0 0 0"/>
+        <mass value="2.43"/>
+        <inertia ixx="0.3" ixy="0.0" ixz="0.0" iyy="0.3" iyz="0.0" izz="0.3"/>
+      </inertial>
     </link>
     <joint name="${arm_id}_joint4" type="revolute">
@@ -161,7 +136,5 @@
       <axis xyz="0 0 1"/>
       <limit effort="87" lower="-3.0718" upper="-0.0698" velocity="2.1750"/>
-      <!-- for simulation -->
-      <dynamics damping="${joint_damping}"/>
-      <!-- end for simulation -->
+      <dynamics damping="${joint_damping}"/>
     </joint>
     <link name="${arm_id}_link5">
@@ -176,13 +149,9 @@
         </geometry>
       </collision>
-      <!-- for simulation -->
-        <!-- Link 5 -->
-        <!-- Generated From:  git@github.com:marcocognetti/FrankaEmikaPandaDynModel.git -->
-        <inertial>
-            <origin xyz="-0.000323 0.021146 -0.124488" rpy="0 0 0" />
-            <mass value="2.095362"/>
-            <inertia  ixx="0.025776" ixy="0.003369" ixz="-0.010502" iyy="0.034795" iyz="0.002025" izz="0.000000"  />
-        </inertial>
-      <!-- end for simulation -->
+      <inertial>
+        <origin xyz="0 0 0" rpy="0 0 0"/>
+        <mass value="3.5"/>
+        <inertia ixx="0.3" ixy="0.0" ixz="0.0" iyy="0.3" iyz="0.0" izz="0.3"/>
+      </inertial>
     </link>
     <joint name="${arm_id}_joint5" type="revolute">
@@ -193,7 +162,5 @@
       <axis xyz="0 0 1"/>
       <limit effort="12" lower="-2.8973" upper="2.8973" velocity="2.6100"/>
-      <!-- for simulation -->
-      <dynamics damping="${joint_damping}"/>
-      <!-- end for simulation -->
+      <dynamics damping="${joint_damping}"/>
     </joint>
     <link name="${arm_id}_link6">
@@ -208,13 +175,9 @@
         </geometry>
       </collision>
-      <!-- for simulation -->
-        <!-- Link 6 -->
-        <!-- Generated From:  git@github.com:marcocognetti/FrankaEmikaPandaDynModel.git -->
-        <inertial>
-            <origin xyz="0.066189 -0.018040 -0.021379" rpy="0 0 0" />
-            <mass value="1.722535"/>
-            <inertia  ixx="0.000104" ixy="-0.003459" ixz="0.002509" iyy="0.003188" iyz="0.001801" izz="0.000622"  />
-        </inertial>
-      <!-- end for simulation -->
+      <inertial>
+        <origin xyz="0 0 0" rpy="0 0 0"/>
+        <mass value="1.47"/>
+        <inertia ixx="0.3" ixy="0.0" ixz="0.0" iyy="0.3" iyz="0.0" izz="0.3"/>
+      </inertial>
     </link>
     <joint name="${arm_id}_joint6" type="revolute">
@@ -225,7 +188,5 @@
       <axis xyz="0 0 1"/>
       <limit effort="12" lower="-0.0175" upper="3.7525" velocity="2.6100"/>
-      <!-- for simulation -->
-      <dynamics damping="${joint_damping}"/>
-      <!-- end for simulation -->
+      <dynamics damping="${joint_damping}"/>
     </joint>
     <link name="${arm_id}_link7">
@@ -240,13 +201,9 @@
         </geometry>
       </collision>
-      <!-- for simulation -->
-        <!-- Link 7 -->
-        <!-- Generated From:  git@github.com:marcocognetti/FrankaEmikaPandaDynModel.git -->
-        <inertial>
-            <origin xyz="0.001859 0.007351 0.055465" rpy="0 0 0" />
-            <mass value="0.570636"/>
-            <inertia  ixx="0.002852" ixy="0.004632" ixz="0.002398" iyy="0.000000" iyz="-0.002696" izz="0.000000"  />
-        </inertial>
-      <!-- end for simulation -->
+      <inertial>
+        <origin xyz="0 0 0" rpy="0 0 0"/>
+        <mass value="0.45"/>
+        <inertia ixx="0.3" ixy="0.0" ixz="0.0" iyy="0.3" iyz="0.0" izz="0.3"/>
+      </inertial>
     </link>
     <joint name="${arm_id}_joint7" type="revolute">
@@ -257,16 +214,12 @@
       <axis xyz="0 0 1"/>
       <limit effort="12" lower="-2.8973" upper="2.8973" velocity="2.6100"/>
-      <!-- for simulation -->
-      <dynamics damping="${joint_damping}"/>
-      <!-- end for simulation -->
+      <dynamics damping="${joint_damping}"/>
     </joint>
     <link name="${arm_id}_link8">
-      <!-- for simulation -->
-      <inertial>
-        <origin xyz="0 0 0" rpy="0 0 0" />
-        <mass value="0.0" />
-        <inertia ixx="0.3" ixy="0.0" ixz="0.0" iyy="0.3" iyz="0.0" izz="0.3" />
-      </inertial>
-      <!-- end for simulation -->
+      <inertial>
+        <origin xyz="0 0 0" rpy="0 0 0"/>
+        <mass value="0.0"/>
+        <inertia ixx="0.3" ixy="0.0" ixz="0.0" iyy="0.3" iyz="0.0" izz="0.3"/>
+      </inertial>
     </link>
     <joint name="${arm_id}_joint8" type="fixed">

Commit message: Remove 0 inertias

File: franka_description/robots/panda_arm.xacro (robot description, xacro)
@@ -118,5 +118,5 @@
             <origin xyz="0.032833 -0.002029 -0.096799" rpy="0 0 0" />
             <mass value="3.300138"/>
-            <inertia  ixx="0.035301" ixy="0.011494" ixz="-0.016618" iyy="0.003726" iyz="-0.013031" izz="0.000000"  />
+            <inertia  ixx="0.035301" ixy="0.011494" ixz="-0.016618" iyy="0.003726" iyz="-0.013031" izz="0.0001"  />
         </inertial>
       <!-- end for simulation -->
@@ -150,5 +150,5 @@
             <origin xyz="-0.043407 0.128195 0.002060" rpy="0 0 0" />
             <mass value="2.548403"/>
-            <inertia  ixx="0.022739" ixy="-0.011128" ixz="0.003843" iyy="0.000000" iyz="0.007803" izz="0.028460"  />
+            <inertia  ixx="0.022739" ixy="-0.011128" ixz="0.003843" iyy="0.0001" iyz="0.007803" izz="0.028460"  />
         </inertial>
       <!-- end for simulation -->
@@ -182,5 +182,5 @@
             <origin xyz="-0.000323 0.021146 -0.124488" rpy="0 0 0" />
             <mass value="2.095362"/>
-            <inertia  ixx="0.025776" ixy="0.003369" ixz="-0.010502" iyy="0.034795" iyz="0.002025" izz="0.000000"  />
+            <inertia  ixx="0.025776" ixy="0.003369" ixz="-0.010502" iyy="0.034795" iyz="0.002025" izz="0.0001"  />
         </inertial>
       <!-- end for simulation -->
@@ -246,5 +246,5 @@
             <origin xyz="0.001859 0.007351 0.055465" rpy="0 0 0" />
             <mass value="0.570636"/>
-            <inertia  ixx="0.002852" ixy="0.004632" ixz="0.002398" iyy="0.000000" iyz="-0.002696" izz="0.000000"  />
+            <inertia  ixx="0.002852" ixy="0.004632" ixz="0.002398" iyy="0.0001" iyz="-0.002696" izz="0.0001"  />
         </inertial>
       <!-- end for simulation -->
