Commit message: Reduce M and inertias

File: franka_description/robots/hand.xacro (robot description, xacro)
@@ -25,5 +25,5 @@
         <origin xyz="0 0 0" rpy="0 0 0" />
         <mass value="0.68" />
-        <inertia ixx="0.1" ixy="0.0" ixz="0.0" iyy="0.1" iyz="0.0" izz="0.1" />
+        <inertia ixx="0.01" ixy="0.0" ixz="0.0" iyy="0.01" iyz="0.0" izz="0.01" />
       </inertial>
       <!-- end for simulation -->
@@ -44,5 +44,5 @@
         <origin xyz="0 0 0" rpy="0 0 0" />
         <mass value="0.01" />
-        <inertia ixx="0.1" ixy="0.0" ixz="0.0" iyy="0.1" iyz="0.0" izz="0.1" />
+        <inertia ixx="0.0001" ixy="0.0" ixz="0.0" iyy="0.0001" iyz="0.0" izz="0.0001" />
       </inertial>
       <!-- end for simulation -->
@@ -65,5 +65,5 @@
         <origin xyz="0 0 0" rpy="0 0 0" />
         <mass value="0.01" />
-        <inertia ixx="0.1" ixy="0.0" ixz="0.0" iyy="0.1" iyz="0.0" izz="0.1" />
+        <inertia ixx="0.0001" ixy="0.0" ixz="0.0" iyy="0.0001" iyz="0.0" izz="0.0001" />
       </inertial>
       <!-- end for simulation -->

File: franka_description/robots/panda.gazebo.xacro (robot description, xacro)
@@ -2,15 +2,17 @@
 <robot xmlns:xacro="http://www.ros.org/wiki/xacro">
     <xacro:macro name="panda_gazebo" params="robot_name">
+        <xacro:property name="mu1" value="0.0"/>
+        <xacro:property name="mu2" value="0.0"/>
         <!-- Link0 -->
         <gazebo reference="${robot_name}_link0">
             <!-- <material>Gazebo/Grey</material> -->
-            <mu1>0.2</mu1>
-            <mu2>0.2</mu2>
+            <mu1>${mu1}</mu1>
+            <mu2>${mu2}</mu2>
         </gazebo>
         <!-- Link1 -->
         <gazebo reference="${robot_name}_link1">
             <!-- <material>Gazebo/White</material> -->
-            <mu1>0.2</mu1>
-            <mu2>0.2</mu2>
+            <mu1>${mu1}</mu1>
+            <mu2>${mu2}</mu2>
         </gazebo>
         <!-- Link2 -->
@@ -23,54 +25,54 @@
         <gazebo reference="${robot_name}_link3">
             <!-- <material>Gazebo/White</material> -->
-            <mu1>0.2</mu1>
-            <mu2>0.2</mu2>
+            <mu1>${mu1}</mu1>
+            <mu2>${mu2}</mu2>
         </gazebo>
         <!-- Link4 -->
         <gazebo reference="${robot_name}_link4">
             <!-- <material>Gazebo/White</material> -->
-            <mu1>0.2</mu1>
-            <mu2>0.2</mu2>
+            <mu1>${mu1}</mu1>
+            <mu2>${mu2}</mu2>
         </gazebo>
         <!-- Link5 -->
         <gazebo reference="${robot_name}_link5">
             <!-- <material>Gazebo/White</material> -->
-            <mu1>0.2</mu1>
-            <mu2>0.2</mu2>
+            <mu1>${mu1}</mu1>
+            <mu2>${mu2}</mu2>
         </gazebo>
         <!-- Link6 -->
         <gazebo reference="${robot_name}_link6">
             <!-- <material>Gazebo/White</material> -->
-            <mu1>0.2</mu1>
-            <mu2>0.2</mu2>
+            <mu1>${mu1}</mu1>
+            <mu2>${mu2}</mu2>
         </gazebo>
         <!-- Link7 -->
         <gazebo reference="${robot_name}_link7">
             <!-- <material>Gazebo/Grey</material> -->
-            <mu1>0.2</mu1>
-            <mu2>0.2</mu2>
+            <mu1>${mu1}</mu1>
+            <mu2>${mu2}</mu2>
         </gazebo>
         <!-- Link8 -->
         <gazebo reference="${robot_name}_link8">
             <!-- <material>Gazebo/Grey</material> -->
-            <mu1>0.2</mu1>
-            <mu2>0.2</mu2>
+            <mu1>${mu1}</mu1>
+            <mu2>${mu2}</mu2>
         </gazebo>
         <!-- LinkHand -->
         <gazebo reference="${robot_name}_hand">
             <!-- <material>Gazebo/Grey</material> -->
-            <mu1>0.2</mu1>
-            <mu2>0.2</mu2>
+            <mu1>${mu1}</mu1>
+            <mu2>${mu2}</mu2>
         </gazebo>
         <!-- LinkRightFinger -->
         <gazebo reference="${robot_name}_rightfinger">
             <!-- <material>Gazebo/Grey</material> -->
-            <mu1>0.2</mu1>
-            <mu2>0.2</mu2>
+            <mu1>${mu1}</mu1>
+            <mu2>${mu2}</mu2>
         </gazebo>
         <!-- LinkLeftFinger -->
         <gazebo reference="${robot_name}_leftfinger">
             <!-- <material>Gazebo/Grey</material> -->
-            <mu1>0.2</mu1>
-            <mu2>0.2</mu2>
+            <mu1>${mu1}</mu1>
+            <mu2>${mu2}</mu2>
         </gazebo>
     </xacro:macro>

File: franka_description/robots/panda_arm.xacro (robot description, xacro)
@@ -16,5 +16,5 @@
       <origin xyz="0.0 0.0 0.0" rpy="0.0 0.0 0.0" />
     </joint>
-    <xacro:property name="joint_damping" value="1.0"/>
+    <xacro:property name="joint_damping" value="0.0"/>
     <!-- end for simulation -->
     <link name="${arm_id}_link0">
@@ -24,9 +24,9 @@
         </geometry>
       </visual>
-      <collision>
+      <!--<collision>
         <geometry>
           <mesh filename="package://${description_pkg}/meshes/collision/link0.stl"/>
         </geometry>
-      </collision>
+      </collision>-->
       <!-- for simulation -->
       <inertial>
@@ -43,9 +43,9 @@
         </geometry>
       </visual>
-      <collision>
+      <!--<collision>
         <geometry>
           <mesh filename="package://${description_pkg}/meshes/collision/link1.stl"/>
         </geometry>
-      </collision>
+      </collision>-->
       <!-- for simulation -->
       <!-- Link 1 -->
@@ -59,5 +59,5 @@
     </link>
     <joint name="${arm_id}_joint1" type="revolute">
-      <safety_controller k_position="100.0" k_velocity="40.0" soft_lower_limit="-2.8973" soft_upper_limit="2.8973"/>
+      <!--<safety_controller k_position="100.0" k_velocity="40.0" soft_lower_limit="-2.8973" soft_upper_limit="2.8973"/>-->
       <origin rpy="0 0 0" xyz="0 0 0.333"/>
       <parent link="${arm_id}_link0"/>
@@ -66,5 +66,5 @@
       <limit effort="87" lower="-2.8973" upper="2.8973" velocity="2.1750"/>
       <!-- for simulation -->
-      <dynamics damping="${joint_damping}"/>
+      <!--<dynamics damping="${joint_damping}"/>-->
       <!-- end for simulation -->
     </joint>
@@ -75,9 +75,9 @@
         </geometry>
       </visual>
-      <collision>
+      <!--<collision>
         <geometry>
           <mesh filename="package://${description_pkg}/meshes/collision/link2.stl"/>
         </geometry>
-      </collision>
+      </collision>-->
       <!-- for simulation -->
         <!-- Link 2 -->
@@ -91,5 +91,5 @@
     </link>
     <joint name="${arm_id}_joint2" type="revolute">
-      <safety_controller k_position="100.0" k_velocity="40.0" soft_lower_limit="-1.7628" soft_upper_limit="1.7628"/>
+      <!--<safety_controller k_position="100.0" k_velocity="40.0" soft_lower_limit="-1.7628" soft_upper_limit="1.7628"/>-->
       <origin rpy="${-pi/2} 0 0" xyz="0 0 0"/>
       <parent link="${arm_id}_link1"/>
@@ -98,5 +98,5 @@
       <limit effort="87" lower="-1.7628" upper="1.7628" velocity="2.1750"/>
       <!-- for simulation -->
-      <dynamics damping="${joint_damping}"/>
+      <!--<dynamics damping="${joint_damping}"/>-->
       <!-- end for simulation -->
     </joint>
@@ -107,9 +107,9 @@
         </geometry>
       </visual>
-      <collision>
+      <!--<collision>
         <geometry>
           <mesh filename="package://${description_pkg}/meshes/collision/link3.stl"/>
         </geometry>
-      </collision>
+      </collision>-->
       <!-- for simulation -->
         <!-- Link 3 -->
@@ -123,5 +123,5 @@
     </link>
     <joint name="${arm_id}_joint3" type="revolute">
-      <safety_controller k_position="100.0" k_velocity="40.0" soft_lower_limit="-2.8973" soft_upper_limit="2.8973"/>
+      <!--<safety_controller k_position="100.0" k_velocity="40.0" soft_lower_limit="-2.8973" soft_upper_limit="2.8973"/>-->
       <origin rpy="${pi/2} 0 0" xyz="0 -0.316 0"/>
       <parent link="${arm_id}_link2"/>
@@ -130,5 +130,5 @@
       <limit effort="87" lower="-2.8973" upper="2.8973" velocity="2.1750"/>
       <!-- for simulation -->
-      <dynamics damping="${joint_damping}"/>
+      <!--<dynamics damping="${joint_damping}"/>-->
       <!-- end for simulation -->
     </joint>
@@ -139,9 +139,9 @@
         </geometry>
       </visual>
-      <collision>
+      <!--<collision>
         <geometry>
           <mesh filename="package://${description_pkg}/meshes/collision/link4.stl"/>
         </geometry>
-      </collision>
+      </collision>-->
       <!-- for simulation -->
         <!-- Link 4 -->
@@ -155,5 +155,5 @@
     </link>
     <joint name="${arm_id}_joint4" type="revolute">
-      <safety_controller k_position="100.0" k_velocity="40.0" soft_lower_limit="-3.0718" soft_upper_limit="-0.0698"/>
+      <!--<safety_controller k_position="100.0" k_velocity="40.0" soft_lower_limit="-3.0718" soft_upper_limit="-0.0698"/>-->
       <origin rpy="${pi/2} 0 0" xyz="0.0825 0 0"/>
       <parent link="${arm_id}_link3"/>
@@ -162,5 +162,5 @@
       <limit effort="87" lower="-3.0718" upper="-0.0698" velocity="2.1750"/>
       <!-- for simulation -->
-      <dynamics damping="${joint_damping}"/>
+      <!--<dynamics damping="${joint_damping}"/>-->
       <!-- end for simulation -->
     </joint>
@@ -171,9 +171,9 @@
         </geometry>
       </visual>
-      <collision>
+      <!--<collision>
         <geometry>
           <mesh filename="package://${description_pkg}/meshes/collision/link5.stl"/>
         </geometry>
-      </collision>
+      </collision>-->
       <!-- for simulation -->
         <!-- Link 5 -->
@@ -187,5 +187,5 @@
     </link>
     <joint name="${arm_id}_joint5" type="revolute">
-      <safety_controller k_position="100.0" k_velocity="40.0" soft_lower_limit="-2.8973" soft_upper_limit="2.8973"/>
+      <!--<safety_controller k_position="100.0" k_velocity="40.0" soft_lower_limit="-2.8973" soft_upper_limit="2.8973"/>-->
       <origin rpy="${-pi/2} 0 0" xyz="-0.0825 0.384 0"/>
       <parent link="${arm_id}_link4"/>
@@ -194,5 +194,5 @@
       <limit effort="12" lower="-2.8973" upper="2.8973" velocity="2.6100"/>
       <!-- for simulation -->
-      <dynamics damping="${joint_damping}"/>
+      <!--<dynamics damping="${joint_damping}"/>-->
       <!-- end for simulation -->
     </joint>
@@ -203,9 +203,9 @@
         </geometry>
       </visual>
-      <collision>
+      <!--<collision>
         <geometry>
           <mesh filename="package://${description_pkg}/meshes/collision/link6.stl"/>
         </geometry>
-      </collision>
+      </collision>-->
       <!-- for simulation -->
         <!-- Link 6 -->
@@ -219,5 +219,5 @@
     </link>
     <joint name="${arm_id}_joint6" type="revolute">
-      <safety_controller k_position="100.0" k_velocity="40.0" soft_lower_limit="-0.0175" soft_upper_limit="3.7525"/>
+      <!--<safety_controller k_position="100.0" k_velocity="40.0" soft_lower_limit="-0.0175" soft_upper_limit="3.7525"/>-->
       <origin rpy="${pi/2} 0 0" xyz="0 0 0"/>
       <parent link="${arm_id}_link5"/>
@@ -226,5 +226,5 @@
       <limit effort="12" lower="-0.0175" upper="3.7525" velocity="2.6100"/>
       <!-- for simulation -->
-      <dynamics damping="${joint_damping}"/>
+      <!--<dynamics damping="${joint_damping}"/>-->
       <!-- end for simulation -->
     </joint>
@@ -235,9 +235,9 @@
         </geometry>
       </visual>
-      <collision>
+      <!--<collision>
         <geometry>
           <mesh filename="package://${description_pkg}/meshes/collision/link7.stl"/>
         </geometry>
-      </collision>
+      </collision>-->
       <!-- for simulation -->
         <!-- Link 7 -->
@@ -251,5 +251,5 @@
     </link>
     <joint name="${arm_id}_joint7" type="revolute">
-      <safety_controller k_position="100.0" k_velocity="40.0" soft_lower_limit="-2.8973" soft_upper_limit="2.8973"/>
+      <!--<safety_controller k_position="100.0" k_velocity="40.0" soft_lower_limit="-2.8973" soft_upper_limit="2.8973"/>-->
       <origin rpy="${pi/2} 0 0" xyz="0.088 0 0"/>
       <parent link="${arm_id}_link6"/>
@@ -258,5 +258,5 @@
       <limit effort="12" lower="-2.8973" upper="2.8973" velocity="2.6100"/>
       <!-- for simulation -->
-      <dynamics damping="${joint_damping}"/>
+      <!--<dynamics damping="${joint_damping}"/>-->
       <!-- end for simulation -->
     </joint>
@@ -266,5 +266,5 @@
         <origin xyz="0 0 0" rpy="0 0 0" />
         <mass value="0.0" />
-        <inertia ixx="0.3" ixy="0.0" ixz="0.0" iyy="0.3" iyz="0.0" izz="0.3" />
+        <inertia ixx="0.0" ixy="0.0" ixz="0.0" iyy="0.0" iyz="0.0" izz="0.0" />
       </inertial>
       <!-- end for simulation -->
